Commit message: Fix Zero USV model frame orientation

File: ros2_ws/src/zero_description/urdf/robot.urdf (robot description, URDF)
Before this commit: robot zero_usv, 4 links, 3 joints
Joints:
- joint left_motor_fixed_joint: origin xyz=0.202 0.111 0.04 rpy=1.5708 0 1.5708 -> xyz=-0.111 0.202 0.04 rpy=1.5708 0 3.1416
- joint right_motor_fixed_joint: origin xyz=-0.205 0.111 0.04 rpy=1.5708 0 1.5708 -> xyz=-0.111 -0.205 0.04 rpy=1.5708 0 3.1416
- joint zero_lidar_fixed_joint: origin xyz=-0.00040397 0.00015 0.1277 rpy=3.1416 0 1.5708 -> xyz=-0.00015 -0.00040397 0.1277 rpy=3.1416 0 3.1416

Commit message: Align Zero USV child link frames

File: ros2_ws/src/zero_description/urdf/robot.urdf (robot description, URDF)
Before this commit: robot zero_usv, 4 links, 3 joints
Joints:
- joint left_motor_fixed_joint: origin xyz=-0.111 0.202 0.04 rpy=1.5708 0 3.1416 -> xyz=-0.111 0.202 0.04 rpy=0 0 0
- joint right_motor_fixed_joint: origin xyz=-0.111 -0.205 0.04 rpy=1.5708 0 3.1416 -> xyz=-0.111 -0.205 0.04 rpy=0 0 0
- joint zero_lidar_fixed_joint: origin xyz=-0.00015 -0.00040397 0.1277 rpy=3.1416 0 3.1416 -> xyz=-0.00015 -0.00040397 0.1277 rpy=0 0 0

Commit message: Add zero_description sensor frame contracts

File: ros2_ws/src/zero_description/urdf/robot.urdf (robot description, URDF)
Before this commit: robot zero_usv, 4 links, 3 joints
Links:
- added link imu_link
- added link laser_frame
Joints:
- added joint zero_imu_fixed_joint: type fixed, parent zero_base_link, child imu_link, origin xyz=0.15 0 0.13 rpy=0 0 0
- added joint zero_laser_frame_fixed_joint: type fixed, parent lidar_link, child laser_frame, origin xyz=0 0 0 rpy=0 0 0
